File: Hardware/0. Project/StreamDeck.brd (EAGLE design)
At the start: 160 x 100 mm, 28 parts, among them SW1 CHERRY_MX, SW10 CHERRY_MX, SW11 CHERRY_MX, SW12 CHERRY_MX, SW2 CHERRY_MX, SW3 CHERRY_MX, SW4 CHERRY_MX, SW5 CHERRY_MX, SW6 CHERRY_MX, SW7 CHERRY_MX, SW8 CHERRY_MX, SW9 CHERRY_MX

Commit message: Schematic WIP
Parts:
- added C1: 10uF, My-RLC:C0805
- added C10, C11, C12, C13, C14, C15, C16, C17, C18, C19, C20, C4, C6, C7, C8, C9: 100nF, My-RLC:C0603
- added C3, C5: 1uF, My-RLC:C0603
- added CN1: Micro USB Type B, My-Connectors:10118193-0001LF
- added CN2: 3.7V, My-Battery:JST-PH2
- added D13, D14: SS34, My-Diodes:DO214AB
- added LED1, LED10, LED11, LED12, LED2, LED3, LED4, LED5, LED6, LED7, LED8, LED9: WS2812B, My-LED:5050
- added R10, R9: 220k (5%), My-RLC:R0603
- added R4: 150R, My-RLC:R0603
- added R5, R7: 22R (5%), My-RLC:R0603
- added R8: 10k (5%), My-RLC:R0603
- added U2: ATMEGA32U4, SparkFun_Pro_Micro_v13a:TESTING_QFN-44
- added Y1: 16MHz, crystal-geyer_V1_0:5.0X3.2_KX-9A
- R1, R2, R3, R6: value (none) -> SLIDE-POT; device rcl:PT-10S -> My-Potentiometers:SLIDER-75MM
- moved R3 298.6 mm to (95.6, 14.6)
- moved R2 295.3 mm to (106.7, 14.6)
- moved R1 292.9 mm to (118.1, 14.6)
- moved R6 269.7 mm to (84.5, 14.6)
- moved D12 222.7 mm to (66.0, 37.8), flipped to the bottom
- moved D11 219.8 mm to (49.5, 37.8), flipped to the bottom
- moved SW12 194.0 mm to (70.5, 31.8)
- moved D10 193.0 mm to (33.0, 37.8), flipped to the bottom
- moved D9 192.7 mm to (16.5, 37.8), flipped to the bottom
- moved D8 181.7 mm to (66.0, 55.6), flipped to the bottom
- moved D7 178.9 mm to (49.5, 55.6), flipped to the bottom
- moved D6 176.5 mm to (33.0, 55.6), flipped to the bottom
- moved D5 174.5 mm to (16.5, 55.6), flipped to the bottom
- moved D4 171.4 mm to (66.0, 73.3), flipped to the bottom
- moved SW7 167.5 mm to (54.0, 49.5)
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Connections:
- new net BATTERY_VOLTAGE: R10.2, R9.2, U2.40
- new net LEDS_CONTROL: LED1.4-DIN, R4.2
- new net N$10: LED3.2-DOUT, LED4.4-DIN
- new net N$15: LED2.2-DOUT, LED3.4-DIN
- new net N$16: LED5.2-DOUT, LED6.4-DIN
- new net N$17: LED6.2-DOUT, LED7.4-DIN
- new net N$18: LED4.2-DOUT, LED5.4-DIN
- new net N$19: LED8.2-DOUT, LED9.4-DIN
- new net N$20: LED10.2-DOUT, LED11.4-DIN
- new net N$21: LED10.4-DIN, LED9.2-DOUT
- new net N$22: LED11.2-DOUT, LED12.4-DIN
- new net N$23: LED7.2-DOUT, LED8.4-DIN
- new net N$24: C5.1, U2.6
- new net N$25: C6.1, U2.42
- new net N$26: C7.1, U2.17, Y1.1
- new net N$27: C8.1, U2.16, Y1.3
- new net N$28: R4.1, U2.29
- new net N$29: R7.2, U2.4
- new net N$30: R5.2, U2.3
- new net N$5: LED1.2-DOUT, LED2.4-DIN
- new net RESET: R8.1, U2.13
- new net USB_D+: CN1.3, R7.1
- new net USB_D-: CN1.2, R5.1
- new net VBAT: CN2.1, D14.A, R10.1
- new net VBUS: C1.1, CN1.1, D13.A, U2.2, U2.7
- net 0V: now also C1.2, C10.2, C11.2, C12.2, C13.2, C14.2, C15.2, C16.2, C17.2, C18.2, C19.2, C20.2, C3.2, C4.2, C5.2, C6.2, C7.2, C8.2, C9.2, CN1.5, CN1.MP1, CN1.MP2, CN1.MP3, CN1.MP4, CN2.2, LED1.3-GND, LED10.3-GND, LED11.3-GND, LED12.3-GND, LED2.3-GND, LED3.3-GND, LED4.3-GND, LED5.3-GND, LED6.3-GND, LED7.3-GND, LED8.3-GND, LED9.3-GND, R1.P$1, R2.P$1, R3.P$1, R6.P$1, R9.1, U2.15, U2.23, U2.33, U2.35, U2.43, U2.5; no longer R1.1, R2.1, R3.1, R6.1
- net 5V: now also C10.1, C11.1, C12.1, C13.1, C14.1, C15.1, C16.1, C17.1, C18.1, C19.1, C20.1, C3.1, C4.1, C9.1, D13.C, D14.C, LED1.1-VDD, LED10.1-VDD, LED11.1-VDD, LED12.1-VDD, LED2.1-VDD, LED3.1-VDD, LED4.1-VDD, LED5.1-VDD, LED6.1-VDD, LED7.1-VDD, LED8.1-VDD, LED9.1-VDD, R1.P$2, R2.P$2, R3.P$2, R6.P$2, R8.2, U2.14, U2.24, U2.34, U2.44; no longer R1.2, R2.2, R3.2, R6.2
- net A0: now also R1.P$6, U2.36; no longer R6.3
- net A1: now also R2.P$6, U2.37; no longer R1.3
- net A2: now also R3.P$6, U2.38; no longer R2.3
- net A3: now also R6.P$6, U2.39; no longer R3.3
- net D2: now also U2.19
- net D3: now also U2.18
- net D4: now also U2.25
- net D5: now also U2.31
- net D6: now also U2.27
- net D7: now also U2.1
- net D8: now also U2.28
Other:
- board size 160 x 100 mm -> 140 x 100 mm
