File: Hardware/0. Project/StreamDeck.sch (EAGLE design)
At the start: 28 parts, among them SW1 CHERRY_MX, SW10 CHERRY_MX, SW11 CHERRY_MX, SW12 CHERRY_MX, SW2 CHERRY_MX, SW3 CHERRY_MX, SW4 CHERRY_MX, SW5 CHERRY_MX, SW6 CHERRY_MX, SW7 CHERRY_MX, SW8 CHERRY_MX, SW9 CHERRY_MX

Commit message: Schematic WIP
Parts:
- added C1: 10uF, My-RLC:C_0805
- added C10, C11, C12, C13, C14, C15, C16, C17, C18, C19, C20, C4, C6, C7, C8, C9: 100nF, My-RLC:C_0603
- added C3, C5: 1uF, My-RLC:C_0603
- added CN1: Micro USB Type B, My-Connectors:MICRO-USB
- added CN2: 3.7V, My-Battery:CELL-CONNECTOR
- added D13, D14: SS34, My-Diodes:SS34
- added LED1, LED10, LED11, LED12, LED2, LED3, LED4, LED5, LED6, LED7, LED8, LED9: WS2812B, My-LED:WS2812B
- added R10, R9: 220k (5%), My-RLC:R_0603
- added R4: 150R, My-RLC:R_0603
- added R5, R7: 22R (5%), My-RLC:R_0603
- added R8: 10k (5%), My-RLC:R_0603
- added U2: ATMEGA32U4, SparkFun_Pro_Micro_v13a:TESTING_ATMEGA32U4QFN
- added Y1: 16MHz, crystal-geyer_V1_0:KX-9A
- R1, R2, R3, R6: value (none) -> SLIDE-POT; device rcl:POTENTIOMETER_PT-10S -> My-Potentiometers:SLIDE-POT
Connections:
- new net BATTERY_VOLTAGE: R10.2, R9.2, U2.PF1(ADC1)
- new net LEDS_CONTROL: LED1.DI, R4.2
- new net N$10: LED3.DO, LED4.DI
- new net N$15: LED2.DO, LED3.DI
- new net N$16: LED5.DO, LED6.DI
- new net N$17: LED6.DO, LED7.DI
- new net N$18: LED4.DO, LED5.DI
- new net N$19: LED8.DO, LED9.DI
- new net N$20: LED10.DO, LED11.DI
- new net N$21: LED10.DI, LED9.DO
- new net N$22: LED11.DO, LED12.DI
- new net N$23: LED7.DO, LED8.DI
- new net N$24: C5.1, U2.UCAP
- new net N$25: C6.1, U2.AREF
- new net N$26: C7.1, U2.XTAL1, Y1.1
- new net N$27: C8.1, U2.XTAL2, Y1.2
- new net N$28: R4.1, U2.PB5(ADC12)
- new net N$29: R7.2, U2.D+
- new net N$30: R5.2, U2.D-
- new net N$5: LED1.DO, LED2.DI
- new net RESET: R8.1, U2.!RESET
- new net USB_D+: CN1G$1.3, R7.1
- new net USB_D-: CN1G$1.2, R5.1
- new net VBAT: CN2.+, D14.A, R10.1
- new net VBUS: C1.1, CN1G$1.1, D13.A, U2.UVCC, U2.VBUS
- net 0V: now also C1.2, C10.2, C11.2, C12.2, C13.2, C14.2, C15.2, C16.2, C17.2, C18.2, C19.2, C20.2, C3.2, C4.2, C5.2, C6.2, C7.2, C8.2, C9.2, CN1G$1.5, CN1G$2.S1, CN1G$2.S2, CN1G$2.S3, CN1G$2.S4, CN2.-, LED1.GND, LED10.GND, LED11.GND, LED12.GND, LED2.GND, LED3.GND, LED4.GND, LED5.GND, LED6.GND, LED7.GND, LED8.GND, LED9.GND, R9.1, U2.GND@15, U2.GND@23, U2.GND@35, U2.GND@43, U2.PE2/!HWB, U2.UGND
- net 5V: now also C10.1, C11.1, C12.1, C13.1, C14.1, C15.1, C16.1, C17.1, C18.1, C19.1, C20.1, C3.1, C4.1, C9.1, D13.K, D14.K, LED1.VDD, LED10.VDD, LED11.VDD, LED12.VDD, LED2.VDD, LED3.VDD, LED4.VDD, LED5.VDD, LED6.VDD, LED7.VDD, LED8.VDD, LED9.VDD, R8.2, U2.AVCC@24, U2.AVCC@44, U2.VCC@14, U2.VCC@34
- net A0: now also R1.3, U2.PF7(ADC7); no longer R6.3
- net A1: now also R2.3, U2.PF6(ADC6); no longer R1.3
- net A2: now also R3.3, U2.PF5(ADC5); no longer R2.3
- net A3: now also R6.3, U2.PF4(ADC4); no longer R3.3
- net D2: now also U2.PD1(SDA)
- net D3: now also U2.PD0(SCL)
- net D4: now also U2.PD4(ADC8)
- net D5: now also U2.PC6
- net D6: now also U2.PD7(ADC10)
- net D7: now also U2.PE6
- net D8: now also U2.PB4(ADC11)
Other:
- note added: "1.1"
- note added: "A0"
- note added: "A1"
- note added: "A2"
- note added: "A3"
- note added: "A4"
- note added: "Complete Schematic"
- note added: "D2"
- note added: "D3"
- note added: "D4"
- note added: "D5"
- note added: "D6"
- note added: "D7"
- note added: "D8"
- note added: "D9"
- note added: "Tiago Silva"
- note added: "github.com/TiagoPaulaSilva/ChristmasTree"
- moved on the sheet: D1, D10, D11, D12, D2, D3, D4, D5, D6, D7, D8, D9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
